File: dual_core_foc_micropy.kicad_pcb (KiCad board)
At the start: 2 copper layers, 95 x 95 mm, 67 parts, among them J1 Conn_ARM_SWD_TagConnect_TC203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, J10 xt30, J12 ribbon_2x7_connector, J2 HDMI_A_1.4, J3 Conn_02x04_Odd_Even, J5 ribbon_2x7_connector, J7 qwiic, J8 Conn_01x04, J9 2.54, Q1 HL_S100N85F, U1 DRV8844PWPR, U2 MT6835, U3 INA241, U4 INA241, U5 ADS131M02-TSSOP!!!, U6 MT6701_custom, U7 LM74700, X1 YXC OT2JI 8.192

Commit message: hardware
Parts:
- moved C7 0.60 mm to (84.0, 123.8)
- renumbered C12 to C1, C19 to C10, C20 to C11, C21 to C12, C22 to C13, C10 to C14, C9 to C15, C11 to C16, C14 to C19, C3 to C2, C15 to C20, C16 to C21, C13 to C22, C24 to C23, C25 to C24, C26 to C25, C28 to C26, C29 to C27, C2 to C3, C1 to C4, C4 to C6, C6 to C9, J9 to J1, J10 to J2, J8 to J3, J3 to J4, J7 to J5, J1 to J6, J2 to J7, J5 to J8, J12 to J9, NT2 to NT1, NT1 to NT2, R9 to R1, R5 to R10, R6 to R11, R1 to R2, R10 to R3, R2 to R4, R3 to R5, R4 to R6, R11 to R7, R7 to R8, R8 to R9, U6 to U1, U1 to U2, U2 to U5, U5 to U6
Connections:
- net /drv8844/A1 renamed /A1
- net /drv8844/A2 renamed /A2
- net /drv8844/B1 renamed /B1
- net /drv8844/B2 renamed /B2
- A1 pad D3: /mcu_pico2/SWCLK -> /mcu_pico2/SWDIO
- J6 pad 2: /mcu_pico2/SWCLK -> /mcu_pico2/SWDIO
