File: dual_core_foc_micropy.kicad_sch (KiCad schematic)
At the start: 11 parts, among them J10 xt30, J3 Conn_02x04_Odd_Even, J8 Conn_01x04, J9 2.54, U6 MT6701_custom

Commit message: hardware
Parts:
- added C7: 100u, 1_custom:CHEMI-KE0, symbol Device:C_Polarized_Small
- added J10: 2.54, Connector_PinHeader_2.54mm:PinHeader_1x02_P2.54mm_Vertical, symbol Connector_Generic:Conn_01x02
- renumbered C12 to C1, J9 to J1, J10 to J2, J8 to J3, J3 to J4, U6 to U1
Connections:
- net GND: now also C7.2, J10.2 (Pin_2)
- net Vdrive: now also C7.1, J10.1 (Pin_1)
- net drv8844/A1 renamed A1
- net drv8844/A2 renamed A2
- net drv8844/B1 renamed B1
- net drv8844/B2 renamed B2
Other:
- note added: "1x2 2.54"
- note added: "XT30"
- note added: "drv8844 is rated for 65 volts I want to choose parts that are rated for similar or higher Ill probably never run it close to that high though"
- note added: "i have other boards with this ribbon cable pinout so if this doesnt work i can use other board"
- note added: "incase diode dont work"
- note added: "prevent current flowing back into power supply"
- moved on the sheet: H1, H2, H3, H4, J1, J2, J4
