File: schems/ads131m02.kicad_sch (KiCad schematic)
At the start: 14 parts, among them U5 ADS131M02-TSSOP!!!, X1 YXC OT2JI 8.192

Commit message: hardware
Parts:
- renumbered C14 to C19, C15 to C20, C16 to C21, C13 to C22, NT1 to NT2, R5 to R10, R6 to R11, R7 to R8, R8 to R9, U5 to U6
Changed lines of the file:
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@@
 				(thickness 0.762)
 				(bold yes)
-				(color 255 255 194 1)
+				(color 0 0 255 1)
 			)
 		)
@@
 		(dnp no)
 		(fields_autoplaced yes)
-		(property "Reference" "#PWR033"
+		(property "Reference" "#PWR042"
 			(at 168.91 80.01 0)
 			(hide yes)
@@
 			(project "dual_core_foc_micropy"
 				(path "/d214fd6e-2db0-437c-9688-cb5c4049811c/c285e8e9-5807-4803-93c1-c03e4e6c8e02"
-					(reference "#PWR033")
+					(reference "#PWR042")
 					(unit 1)
 				)
@@
 		(in_pos_files yes)
 		(dnp no)
-		(property "Reference" "C14"
+		(property "Reference" "C19"
 			(at 135.636 72.898 0)
 			(show_name no)
@@
 			(project "dual_core_foc_micropy"
 				(path "/d214fd6e-2db0-437c-9688-cb5c4049811c/c285e8e9-5807-4803-93c1-c03e4e6c8e02"
-					(reference "C14")
+					(reference "C19")
 					(unit 1)
 				)
@@
 		(dnp no)
 		(fields_autoplaced yes)
-		(property "Reference" "#PWR038"
+		(property "Reference" "#PWR039"
 			(at 152.4 130.81 0)
 			(hide yes)
@@
 			(project "dual_core_foc_micropy"
 				(path "/d214fd6e-2db0-437c-9688-cb5c4049811c/c285e8e9-5807-4803-93c1-c03e4e6c8e02"
-					(reference "#PWR038")
+					(reference "#PWR039")
 					(unit 1)
 				)
@@
 		(dnp no)
 		(fields_autoplaced yes)
-		(property "Reference" "#PWR035"
+		(property "Reference" "#PWR037"
 			(at 144.78 66.04 0)
 			(hide yes)
@@
 			(project "dual_core_foc_micropy"
 				(path "/d214fd6e-2db0-437c-9688-cb5c4049811c/c285e8e9-5807-4803-93c1-c03e4e6c8e02"
-					(reference "#PWR035")
+					(reference "#PWR037")
 					(unit 1)
 				)
@@
 		(dnp no)
 		(fields_autoplaced yes)
-		(property "Reference" "#PWR036"
+		(property "Reference" "#PWR038"
 			(at 151.13 77.47 0)
 			(hide yes)
@@
 			(project "dual_core_foc_micropy"
 				(path "/d214fd6e-2db0-437c-9688-cb5c4049811c/c285e8e9-5807-4803-93c1-c03e4e6c8e02"
-					(reference "#PWR036")
+					(reference "#PWR038")
 					(unit 1)
 				)
@@
 		(dnp no)
 		(fields_autoplaced yes)
-		(property "Reference" "#PWR040"
+		(property "Reference" "#PWR041"
 			(at 165.1 130.81 0)
 			(hide yes)
@@
 			(project "dual_core_foc_micropy"
 				(path "/d214fd6e-2db0-437c-9688-cb5c4049811c/c285e8e9-5807-4803-93c1-c03e4e6c8e02"
-					(reference "#PWR040")
+					(reference "#PWR041")
 					(unit 1)
 				)
@@
 		(in_pos_files yes)
 		(dnp no)
-		(property "Reference" "C13"
+		(property "Reference" "C22"
 			(at 163.576 67.818 0)
 			(show_name no)
@@
 			(project "dual_core_foc_micropy"
 				(path "/d214fd6e-2db0-437c-9688-cb5c4049811c/c285e8e9-5807-4803-93c1-c03e4e6c8e02"
-					(reference "C13")
+					(reference "C22")
 					(unit 1)
 				)
@@
 		(in_pos_files yes)
 		(dnp no)
-		(property "Reference" "R7"
+		(property "Reference" "R8"
 			(at 101.6 90.17 90)
 			(show_name no)
@@
 			(project "dual_core_foc_micropy"
 				(path "/d214fd6e-2db0-437c-9688-cb5c4049811c/c285e8e9-5807-4803-93c1-c03e4e6c8e02"
-					(reference "R7")
+					(reference "R8")
 					(unit 1)
 				)
@@
 		(dnp no)
 		(fields_autoplaced yes)
-		(property "Reference" "#PWR032"
+		(property "Reference" "#PWR043"
 			(at 177.8 69.85 0)
 			(hide yes)
@@
 			(project "dual_core_foc_micropy"
 				(path "/d214fd6e-2db0-437c-9688-cb5c4049811c/c285e8e9-5807-4803-93c1-c03e4e6c8e02"
-					(reference "#PWR032")
+					(reference "#PWR043")
 					(unit 1)
 				)
@@
 		(dnp no)
 		(fields_autoplaced yes)
-		(property "Reference" "#PWR034"
+		(property "Reference" "#PWR036"
 			(at 140.97 85.09 0)
 			(hide yes)
@@
 			(project "dual_core_foc_micropy"
 				(path "/d214fd6e-2db0-437c-9688-cb5c4049811c/c285e8e9-5807-4803-93c1-c03e4e6c8e02"
-					(reference "#PWR034")
+					(reference "#PWR036")
 					(unit 1)
 				)
@@
 		(in_pos_files yes)
 		(dnp no)
-		(property "Reference" "R6"
+		(property "Reference" "R11"
 			(at 103.886 102.87 90)
 			(show_name no)
@@
 			(project "dual_core_foc_micropy"
 				(path "/d214fd6e-2db0-437c-9688-cb5c4049811c/c285e8e9-5807-4803-93c1-c03e4e6c8e02"
-					(reference "R6")
+					(reference "R11")
 					(unit 1)
 				)
@@
 		(in_pos_files yes)
 		(dnp no)
-		(property "Reference" "R5"
+		(property "Reference" "R10"
 			(at 101.854 100.33 90)
 			(show_name no)
@@
 			(project "dual_core_foc_micropy"
 				(path "/d214fd6e-2db0-437c-9688-cb5c4049811c/c285e8e9-5807-4803-93c1-c03e4e6c8e02"
-					(reference "R5")
+					(reference "R10")
 					(unit 1)
 				)
@@
 		(in_pos_files yes)
 		(dnp no)
-		(property "Reference" "U5"
+		(property "Reference" "U6"
 			(at 135.636 86.868 0)
 			(show_name no)
@@
 			(project "dual_core_foc_micropy"
 				(path "/d214fd6e-2db0-437c-9688-cb5c4049811c/c285e8e9-5807-4803-93c1-c03e4e6c8e02"
-					(reference "U5")
+					(reference "U6")
 					(unit 1)
 				)
@@
 		(dnp no)
 		(fields_autoplaced yes)
-		(property "Reference" "#PWR037"
+		(property "Reference" "#PWR040"
 			(at 156.21 90.17 0)
 			(hide yes)
@@
 			(project "dual_core_foc_micropy"
 				(path "/d214fd6e-2db0-437c-9688-cb5c4049811c/c285e8e9-5807-4803-93c1-c03e4e6c8e02"
-					(reference "#PWR037")
+					(reference "#PWR040")
 					(unit 1)
 				)
@@
 		(in_pos_files yes)
 		(dnp no)
-		(property "Reference" "C16"
+		(property "Reference" "C21"
 			(at 170.434 118.618 0)
 			(show_name no)
@@
 			(project "dual_core_foc_micropy"
 				(path "/d214fd6e-2db0-437c-9688-cb5c4049811c/c285e8e9-5807-4803-93c1-c03e4e6c8e02"
-					(reference "C16")
+					(reference "C21")
 					(unit 1)
 				)
@@
 		(in_pos_files yes)
 		(dnp no)
-		(property "Reference" "C15"
+		(property "Reference" "C20"
 			(at 161.544 77.978 0)
 			(show_name no)
@@
 			(project "dual_core_foc_micropy"
 				(path "/d214fd6e-2db0-437c-9688-cb5c4049811c/c285e8e9-5807-4803-93c1-c03e4e6c8e02"
-					(reference "C15")
+					(reference "C20")
 					(unit 1)
 				)
@@
 		(in_pos_files yes)
 		(dnp no)
-		(property "Reference" "R8"
+		(property "Reference" "R9"
 			(at 103.632 92.71 90)
 			(show_name no)
@@
 			(project "dual_core_foc_micropy"
 				(path "/d214fd6e-2db0-437c-9688-cb5c4049811c/c285e8e9-5807-4803-93c1-c03e4e6c8e02"
-					(reference "R8")
+					(reference "R9")
 					(unit 1)
 				)
@@
 		(dnp no)
 		(fields_autoplaced yes)
-		(property "Reference" "#PWR039"
+		(property "Reference" "#PWR044"
 			(at 177.8 97.79 0)
 			(hide yes)
@@
 			(project "dual_core_foc_micropy"
 				(path "/d214fd6e-2db0-437c-9688-cb5c4049811c/c285e8e9-5807-4803-93c1-c03e4e6c8e02"
-					(reference "#PWR039")
+					(reference "#PWR044")
 					(unit 1)
 				)
@@
 		(in_pos_files yes)
 		(dnp yes)
-		(property "Reference" "NT1"
+		(property "Reference" "NT2"
 			(at 145.796 65.786 90)
 			(show_name no)
@@
 			(project "dual_core_foc_micropy"
 				(path "/d214fd6e-2db0-437c-9688-cb5c4049811c/c285e8e9-5807-4803-93c1-c03e4e6c8e02"
-					(reference "NT1")
+					(reference "NT2")
 					(unit 1)
 				)
