File: schems/drv8844.kicad_sch (KiCad schematic)
At the start: 19 parts, among them U1 DRV8844PWPR, U3 INA241, U4 INA241

Commit message: hardware
Parts:
- removed C7: 100u, 1_custom:CHEMI-KE0, symbol Device:C_Polarized_Small
- renumbered C19 to C10, C20 to C11, C21 to C12, C22 to C13, C10 to C14, C9 to C15, C3 to C2, C2 to C3, C1 to C4, C4 to C6, C6 to C9, R3 to R5, R4 to R6, U1 to U2
Other:
- note added: "+/- flipped for easy routing sig current is bidirectional"
- note removed: "+/- flipped for routing sig current is bidirectional"
