File: schems/ideal_diode.kicad_sch (KiCad schematic)
At the start: 7 parts, among them Q1 HL_S100N85F, U7 LM74700

Commit message: hardware
Parts:
- renumbered C24 to C23, C25 to C24, C26 to C25, C28 to C26, C29 to C27
Other:
- note added: "cathode "atleast 100nf" covered by bulk capacitance (100uf)"
- note added: "vcap gets 15 volts across "vcap > 10 * mosfet C_{iss} in uf" Ciss S100N85F is 4700pf or 4.7nf so 100nf is sufficient"
- note removed: "cathode "atleast 100nf" covered by bulk and drive capacitance"
- note removed: "vcap gets 15 volts across (50v cap ok) "vcap > 10 * mosfet C_{iss} in uf" Ciss S100N85F is 4700pf or 4.7nf so 100nf sufficient"
Changed lines of the file:
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@@
 	(generator_version "10.0")
 	(paper "A4")
-	(text "cathode \"atleast 100nf\"\ncovered by bulk and drive capacitance"
+	(text "cathode \"atleast 100nf\"\ncovered by bulk capacitance (100uf)"
 		(exclude_from_sim no)
-		(at 152.4 67.818 0)
+		(at 177.038 77.47 0)
 		(effects
 			(font
@@
 	(text "\"atleast 22nf input\""
 		(exclude_from_sim no)
-		(at 108.966 95.758 0)
+		(at 123.952 73.152 0)
 		(effects
 			(font
@@
 		)
 	)
-	(text "vcap gets 15 volts across (50v cap ok)\n\"vcap > 10 * mosfet C_{iss} in uf\"\nCiss S100N85F is 4700pf or 4.7nf\nso 100nf sufficient\n\n"
+	(text "vcap gets 15 volts across\n\"vcap > 10 * mosfet C_{iss} in uf\"\nCiss S100N85F is 4700pf or 4.7nf\nso 100nf is sufficient\n\n"
 		(exclude_from_sim no)
-		(at 109.982 121.666 0)
+		(at 102.87 116.84 0)
 		(effects
 			(font
@@
 		(dnp no)
 		(fields_autoplaced yes)
-		(property "Reference" "#PWR052"
+		(property "Reference" "#PWR056"
 			(at 142.24 127 0)
 			(hide yes)
@@
 			(project "dual_core_foc_micropy"
 				(path "/d214fd6e-2db0-437c-9688-cb5c4049811c/8800cac1-8f40-4a73-92eb-69dc9f669b2b"
-					(reference "#PWR052")
+					(reference "#PWR056")
 					(unit 1)
 				)
@@
 		(in_pos_files yes)
 		(dnp no)
-		(property "Reference" "C25"
+		(property "Reference" "C24"
 			(at 118.364 103.632 0)
 			(show_name no)
@@
 			(project "dual_core_foc_micropy"
 				(path "/d214fd6e-2db0-437c-9688-cb5c4049811c/8800cac1-8f40-4a73-92eb-69dc9f669b2b"
-					(reference "C25")
+					(reference "C24")
 					(unit 1)
 				)
@@
 		(in_pos_files yes)
 		(dnp no)
-		(property "Reference" "C24"
+		(property "Reference" "C23"
 			(at 112.522 103.378 0)
 			(show_name no)
@@
 			(project "dual_core_foc_micropy"
 				(path "/d214fd6e-2db0-437c-9688-cb5c4049811c/8800cac1-8f40-4a73-92eb-69dc9f669b2b"
-					(reference "C24")
+					(reference "C23")
 					(unit 1)
 				)
@@
 		(in_pos_files yes)
 		(dnp no)
-		(property "Reference" "C29"
+		(property "Reference" "C27"
 			(at 121.666 85.598 0)
 			(show_name no)
@@
 			(project "dual_core_foc_micropy"
 				(path "/d214fd6e-2db0-437c-9688-cb5c4049811c/8800cac1-8f40-4a73-92eb-69dc9f669b2b"
-					(reference "C29")
+					(reference "C27")
 					(unit 1)
 				)
@@
 		(in_pos_files yes)
 		(dnp no)
-		(property "Reference" "C28"
+		(property "Reference" "C26"
 			(at 121.666 79.248 0)
 			(show_name no)
@@
 			(project "dual_core_foc_micropy"
 				(path "/d214fd6e-2db0-437c-9688-cb5c4049811c/8800cac1-8f40-4a73-92eb-69dc9f669b2b"
-					(reference "C28")
+					(reference "C26")
 					(unit 1)
 				)
@@
 		(in_pos_files yes)
 		(dnp no)
-		(property "Reference" "C26"
+		(property "Reference" "C25"
 			(at 123.444 103.632 0)
 			(show_name no)
@@
 			(project "dual_core_foc_micropy"
 				(path "/d214fd6e-2db0-437c-9688-cb5c4049811c/8800cac1-8f40-4a73-92eb-69dc9f669b2b"
-					(reference "C26")
+					(reference "C25")
 					(unit 1)
 				)
@@
 		(dnp no)
 		(fields_autoplaced yes)
-		(property "Reference" "#PWR059"
+		(property "Reference" "#PWR055"
 			(at 127 97.79 0)
 			(hide yes)
@@
 			(project "dual_core_foc_micropy"
 				(path "/d214fd6e-2db0-437c-9688-cb5c4049811c/8800cac1-8f40-4a73-92eb-69dc9f669b2b"
-					(reference "#PWR059")
+					(reference "#PWR055")
 					(unit 1)
 				)
