File: schems/mcu_pico2.kicad_sch (KiCad schematic)
At the start: 8 parts, among them J1 Conn_ARM_SWD_TagConnect_TC203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, J2 HDMI_A_1.4, J7 qwiic

Commit message: hardware
Parts:
- renumbered J7 to J5, J1 to J6, J2 to J7, R9 to R1, R1 to R2, R10 to R3, R2 to R4
Connections:
- net SWCLK: no longer A1.D3 (SWDIO), J6.2 (SWDIO)
- new net SWDIO: A1.D3 (SWDIO), J6.2 (SWDIO)
Other:
- note added: "if adc doesnt work can use qwiic to connect to one of my i2c load cell boards"
Changed lines of the file:
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@@
+		)
+	)
+	(text "if adc doesnt work \ncan use qwiic to connect to one of my \ni2c load cell boards"
+		(exclude_from_sim no)
+		(at 107.95 173.482 0)
+		(effects
+			(font
+				(size 1.27 1.27)
+			)
 		)
 	)
@@
 	(wire
 		(pts
-			(xy 248.92 177.8) (xy 242.57 177.8)
+			(xy 247.65 177.8) (xy 242.57 177.8)
 		)
 		(stroke
@@
 	(wire
 		(pts
-			(xy 248.92 172.72) (xy 242.57 172.72)
+			(xy 247.65 172.72) (xy 242.57 172.72)
 		)
 		(stroke
@@
 	(wire
 		(pts
-			(xy 252.73 162.56) (xy 242.57 162.56)
+			(xy 247.65 162.56) (xy 242.57 162.56)
 		)
 		(stroke
@@
 	(wire
 		(pts
-			(xy 248.92 175.26) (xy 242.57 175.26)
+			(xy 247.65 175.26) (xy 242.57 175.26)
 		)
 		(stroke
@@
 	(wire
 		(pts
-			(xy 252.73 160.02) (xy 242.57 160.02)
+			(xy 247.65 160.02) (xy 242.57 160.02)
 		)
 		(stroke
@@
 	(wire
 		(pts
-			(xy 252.73 157.48) (xy 242.57 157.48)
+			(xy 247.65 157.48) (xy 242.57 157.48)
 		)
 		(stroke
@@
 		)
 	)
-	(label "SWCLK"
+	(label "SWDIO"
 		(at 182.88 132.08 0)
 		(effects
@@
 	(hierarchical_label "GPIO28"
 		(shape input)
-		(at 248.92 177.8 0)
+		(at 247.65 177.8 0)
 		(effects
 			(font
@@
 	(hierarchical_label "ADC0"
 		(shape input)
-		(at 248.92 172.72 0)
+		(at 247.65 172.72 0)
 		(effects
 			(font
@@
 	(hierarchical_label "PWM2_A"
 		(shape input)
-		(at 252.73 157.48 0)
+		(at 247.65 157.48 0)
 		(effects
 			(font
@@
 	(hierarchical_label "ADC1"
 		(shape input)
-		(at 248.92 175.26 0)
+		(at 247.65 175.26 0)
 		(effects
 			(font
@@
 	(hierarchical_label "GPIO22"
 		(shape input)
-		(at 252.73 162.56 0)
+		(at 247.65 162.56 0)
 		(effects
 			(font
@@
 	(hierarchical_label "PWM2_B"
 		(shape input)
-		(at 252.73 160.02 0)
+		(at 247.65 160.02 0)
 		(effects
 			(font
@@
 		(dnp no)
 		(fields_autoplaced yes)
-		(property "Reference" "#PWR054"
+		(property "Reference" "#PWR07"
 			(at 116.84 156.21 0)
 			(hide yes)
@@
 			(project "dual_core_foc_micropy"
 				(path "/d214fd6e-2db0-437c-9688-cb5c4049811c/15053b24-78c8-4ef8-b22f-7d8e43811ce6"
-					(reference "#PWR054")
+					(reference "#PWR07")
 					(unit 1)
 				)
@@
 		(dnp no)
 		(fields_autoplaced yes)
-		(property "Reference" "#PWR05"
+		(property "Reference" "#PWR015"
 			(at 243.84 198.12 0)
 			(hide yes)
@@
 			(project "dual_core_foc_micropy"
 				(path "/d214fd6e-2db0-437c-9688-cb5c4049811c/15053b24-78c8-4ef8-b22f-7d8e43811ce6"
-					(reference "#PWR05")
+					(reference "#PWR015")
 					(unit 1)
 				)
@@
 		(in_pos_files yes)
 		(dnp no)
-		(property "Reference" "J7"
+		(property "Reference" "J5"
 			(at 103.886 154.686 0)
 			(show_name no)
@@
 			(project "dual_core_foc_micropy"
 				(path "/d214fd6e-2db0-437c-9688-cb5c4049811c/15053b24-78c8-4ef8-b22f-7d8e43811ce6"
-					(reference "J7")
+					(reference "J5")
 					(unit 1)
 				)
@@
 		(in_pos_files yes)
 		(dnp no)
-		(property "Reference" "R1"
+		(property "Reference" "R2"
 			(at 135.89 153.67 90)
 			(show_name no)
@@
 			(project "dual_core_foc_micropy"
 				(path "/d214fd6e-2db0-437c-9688-cb5c4049811c/15053b24-78c8-4ef8-b22f-7d8e43811ce6"
-					(reference "R1")
+					(reference "R2")
 					(unit 1)
 				)
@@
 		(dnp yes)
 		(fields_autoplaced yes)
-		(property "Reference" "J1"
+		(property "Reference" "J6"
 			(at 165.1 128.2699 0)
 			(show_name no)
@@
 			(project "dual_core_foc_micropy"
 				(path "/d214fd6e-2db0-437c-9688-cb5c4049811c/15053b24-78c8-4ef8-b22f-7d8e43811ce6"
-					(reference "J1")
+					(reference "J6")
 					(unit 1)
 				)
@@
 		(in_pos_files yes)
 		(dnp no)
-		(property "Reference" "R2"
+		(property "Reference" "R4"
 			(at 139.7 153.67 90)
 			(show_name no)
@@
 			(project "dual_core_foc_micropy"
 				(path "/d214fd6e-2db0-437c-9688-cb5c4049811c/15053b24-78c8-4ef8-b22f-7d8e43811ce6"
-					(reference "R2")
+					(reference "R4")
 					(unit 1)
 				)
@@
 		(in_pos_files yes)
 		(dnp no)
-		(property "Reference" "R10"
+		(property "Reference" "R3"
 			(at 139.7 147.32 90)
 			(show_name no)
@@
 			(project "dual_core_foc_micropy"
 				(path "/d214fd6e-2db0-437c-9688-cb5c4049811c/15053b24-78c8-4ef8-b22f-7d8e43811ce6"
-					(reference "R10")
+					(reference "R3")
 					(unit 1)
 				)
@@
 		(in_pos_files yes)
 		(dnp no)
-		(property "Reference" "R9"
+		(property "Reference" "R1"
 			(at 135.89 147.32 90)
 			(show_name no)
@@
 			(project "dual_core_foc_micropy"
 				(path "/d214fd6e-2db0-437c-9688-cb5c4049811c/15053b24-78c8-4ef8-b22f-7d8e43811ce6"
-					(reference "R9")
+					(reference "R1")
 					(unit 1)
 				)
@@
 		(in_pos_files no)
 		(dnp no)
-		(fields_autoplaced yes)
 		(property "Reference" "A1"
-			(at 221.8533 194.31 0)
+			(at 200.66 123.952 0)
 			(show_name no)
 			(do_not_autoplace no)
@@
 		)
 		(property "Value" "RaspberryPi_Pico"
-			(at 221.8533 196.85 0)
+			(at 221.742 193.548 0)
 			(show_name no)
 			(do_not_autoplace no)
@@
 		(dnp no)
 		(fields_autoplaced yes)
-		(property "Reference" "#PWR02"
+		(property "Reference" "#PWR011"
 			(at 168.91 148.59 0)
 			(hide yes)
@@
 			(project "dual_core_foc_micropy"
 				(path "/d214fd6e-2db0-437c-9688-cb5c4049811c/15053b24-78c8-4ef8-b22f-7d8e43811ce6"
-					(reference "#PWR02")
+					(reference "#PWR011")
 					(unit 1)
 				)
@@
 		(dnp no)
 		(fields_autoplaced yes)
-		(property "Reference" "#PWR01"
+		(property "Reference" "#PWR010"
 			(at 168.91 120.65 0)
 			(hide yes)
@@
 			(project "dual_core_foc_micropy"
 				(path "/d214fd6e-2db0-437c-9688-cb5c4049811c/15053b24-78c8-4ef8-b22f-7d8e43811ce6"
-					(reference "#PWR01")
+					(reference "#PWR010")
 					(unit 1)
 				)
@@
 		(dnp no)
 		(fields_autoplaced yes)
-		(property "Reference" "#PWR04"
+		(property "Reference" "#PWR013"
 			(at 219.71 207.01 0)
 			(hide yes)
@@
 			(project "dual_core_foc_micropy"
 				(path "/d214fd6e-2db0-437c-9688-cb5c4049811c/15053b24-78c8-4ef8-b22f-7d8e43811ce6"
-					(reference "#PWR04")
+					(reference "#PWR013")
 					(unit 1)
 				)
@@
 		(dnp no)
 		(fields_autoplaced yes)
-		(property "Reference" "#PWR03"
+		(property "Reference" "#PWR012"
 			(at 219.71 114.3 0)
 			(hide yes)
@@
 			(project "dual_core_foc_micropy"
 				(path "/d214fd6e-2db0-437c-9688-cb5c4049811c/15053b24-78c8-4ef8-b22f-7d8e43811ce6"
-					(reference "#PWR03")
+					(reference "#PWR012")
 					(unit 1)
 				)
@@
 		(dnp no)
 		(fields_autoplaced yes)
-		(property "Reference" "#PWR053"
+		(property "Reference" "#PWR08"
 			(at 120.65 162.56 0)
 			(hide yes)
@@
 			(project "dual_core_foc_micropy"
 				(path "/d214fd6e-2db0-437c-9688-cb5c4049811c/15053b24-78c8-4ef8-b22f-7d8e43811ce6"
-					(reference "#PWR053")
+					(reference "#PWR08")
 					(unit 1)
 				)
@@
 		(dnp no)
 		(fields_autoplaced yes)
-		(property "Reference" "#PWR028"
+		(property "Reference" "#PWR09"
 			(at 135.89 146.05 0)
 			(hide yes)
@@
 			(project "dual_core_foc_micropy"
 				(path "/d214fd6e-2db0-437c-9688-cb5c4049811c/15053b24-78c8-4ef8-b22f-7d8e43811ce6"
-					(reference "#PWR028")
+					(reference "#PWR09")
 					(unit 1)
 				)
@@
 		(dnp no)
 		(fields_autoplaced yes)
-		(property "Reference" "#PWR023"
+		(property "Reference" "#PWR014"
 			(at 224.79 114.3 0)
 			(hide yes)
@@
 			(project "dual_core_foc_micropy"
 				(path "/d214fd6e-2db0-437c-9688-cb5c4049811c/15053b24-78c8-4ef8-b22f-7d8e43811ce6"
-					(reference "#PWR023")
+					(reference "#PWR014")
 					(unit 1)
 				)
@@
 		(in_pos_files yes)
 		(dnp no)
-		(property "Reference" "J2"
+		(property "Reference" "J7"
 			(at 313.69 166.3699 0)
 			(show_name no)
@@
 			(project "dual_core_foc_micropy"
 				(path "/d214fd6e-2db0-437c-9688-cb5c4049811c/15053b24-78c8-4ef8-b22f-7d8e43811ce6"
-					(reference "J2")
+					(reference "J7")
 					(unit 1)
 				)
@@
 		(dnp no)
 		(fields_autoplaced yes)
-		(property "Reference" "#PWR06"
+		(property "Reference" "#PWR016"
 			(at 297.18 204.47 0)
 			(hide yes)
@@
 			(project "dual_core_foc_micropy"
 				(path "/d214fd6e-2db0-437c-9688-cb5c4049811c/15053b24-78c8-4ef8-b22f-7d8e43811ce6"
-					(reference "#PWR06")
+					(reference "#PWR016")
 					(unit 1)
 				)
