File: schems/ribbon_cable.kicad_sch (KiCad schematic)
At the start: 2 parts, among them J12 ribbon_2x7_connector, J5 ribbon_2x7_connector

Commit message: hardware
Parts:
- renumbered J5 to J8, J12 to J9
Other:
- note added: "the analog RTD traces are running close to pretty high speed spi. There is 2.5khz RC filter on the ADC though"
- note removed: "yes this is bad to have the analog traces running next to these 10mhz ~50ns or less rise time spi traces however the adc does have pretty heavy (~2.5 or so khz) low pass filtering on its inputs. and this analog reading isnt that critical. not connecting an exc+ and exc- so that i dont couple noise into the more important load cell readings"
- moved on the sheet: J9
