File: schems/snapoff_board.kicad_sch (KiCad schematic)
At the start: 6 parts, among them U2 MT6835

Commit message: hardware
Parts:
- renumbered C11 to C16, NT2 to NT1, R11 to R7, U2 to U5
Other:
- moved on the sheet: NT1, R7, TH1
